File: J0_Drive/_autosave-driver.kicad_sch (KiCad schematic)
At the start: 8 parts, among them J1 Conn_01x02, J2 Conn_01x02, U1 STDRIVE101

Commit message: started VM bulk/decoupling circuit
Parts:
- added C2: 1uF, symbol Device:C
- added C3: 100nF, symbol Device:C
- added TP2: VM, symbol Connector:TestPoint
Connections:
- net GND: now also C2.2, C3.2
- net VS: now reaches U1.4 (VS)
- net REG12: now reaches U1.5 (REG12)
- net nFAULT: now reaches U1.6 (nFAULT)
- new net VM: C2.1, C3.1, TP2.1
Other:
- moved on the sheet: C1, J1, J2, R1, R2, R3, TP1
