File: J0_Drive/halfbridge.kicad_sch (KiCad schematic)
At the start: 13 parts, among them Q1 STL110N10F7, Q2 STL110N10F7, U5 INA240A1PW

Commit message: added CAN and SWD
Parts:
- added NT1: NetTie_2, symbol Device:NetTie_2
Connections:
- net GND: now also NT1.2
- net GNDA: now also NT1.1
- net VDD renamed +3.3V
Other:
- note added: "GNDA will use same ground plane as GND, just grouped separately"
- moved on the sheet: C12, C13, C6, D1, D2, Q1, Q2, R10, R6, R7, R8, R9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

Commit message: organized hierarchical sheets, finished communications, started sensors
Parts:
- renumbered C13 to C15, U5 to U6

Commit message: completed sensing
Parts:
- removed NT1: NetTie_2, symbol Device:NetTie_2
Connections:
- net GNDA is gone; now on net GND: C15.2, U6.1 (GND), U6.4 (GND), U6.7 (REF1)
Other:
- note added: "consider placement for analog"
- note removed: "GNDA will use same ground plane as GND, just grouped separately"
