File: J0_Drive/sensors.kicad_sch (KiCad schematic)
At the start: 1 part, among them U4 AS5047D

Commit message: finished comms SWD header, main page organization
Parts:
- added C18: 4.7u, symbol Device:C
- added C19: 100nF, symbol Device:C
- added TH1: Thermistor_NTC, symbol Device:Thermistor_NTC
Connections:
- net ENC_nCS: now reaches U4.1 (~{CS})
- net ENC_U: now reaches U4.10 (U)
- net +3.3V: now reaches U4.11 (VDD)
- net +3.3V: now also U4.12 (VDD3V3), U4.13 (GND), U4.5 (TST), C18.1, C18.2, C19.1, C19.2
- net ENC_I/PWM: now reaches U4.14 (I/PWM)
- net ENC_CLK: now reaches U4.2 (CLK)
- net ENC_MISO: now reaches U4.3 (MISO)
- net ENC_MOSI: now reaches U4.4 (MOSI)
- net ENC_B: now reaches U4.6 (B)
- net ENC_A: now reaches U4.7 (A)
- net ENC_W/PWM: now reaches U4.8 (W/PWM)
- net ENC_V: now reaches U4.9 (V)
Other:
- note added: "AS5047D (likely will use SPI, have interface for ABI/PWM/UVW"
- note added: "Encoder"
- note added: "Temperature Sensing"
- note added: "Thermistor and voltage divider"

Commit message: completed sensing
Parts:
- added R23: 10k, symbol Device:R
- TH1: value Thermistor_NTC -> 10k
Connections:
- net +3.3V: now also TH1.2, R23.1
- net T_OUT: now reaches TH1.1
- net T_OUT: now also R23.2
Other:
- note added: "Thermistor and voltage divider V_ADC = V_CC * ( R_fixed / ( R_NTC + R_fixed) ) R_NTC = R_fixed * ( ( V_CC / V_ADC ) - 1 R_NTC = 10k * ( ( 3.3 / V_ADC ) - 1 ) 1/T = 1/T_0 + (1/B) * ln ( R / R_0 ) R_0 = 10kOhm (at 25C) T_0 = 298.15K (25C) B = 3950 K TEMP | R_NTC | ADC_V 25C | 10.0k | 1.65 60C | 2.49k | 2.64 80C | 1.27k | 2.93 100C | 0.70k | 3.08"
- note removed: "Thermistor and voltage divider"
- moved on the sheet: TH1
